File: voicecard/hardware_design/pcb/KiCad-SMD/Voicecard-4P-SMD.kicad_sch (KiCad schematic)
At the start: 87 parts, among them IC1 TL074P, IC2 LM13700N, IC3 TL072P, IC4 V2164D, IC5 TL072P, IC6 MCP4822, IC7 ATMega328p, Q1 2N3906, Q2 2N3906, Q3 20MHz

Commit message: Voicecard 4P SMD: assign SMD footprints and LCSC parts in the schematic
Stage A §2 of docs/VOICECARD_SMD_PLAN.md, schematic side only. Each symbol's
Footprint field now names a KiCad standard-library SMD footprint, and every
part JLC will assemble carries an LCSC field. No net and no value changed.

Six Eagle symbols numbered their pins for the through-hole footprint, so the
pin numbers were remapped to the SMD pad numbering: +/- to 1/2 on the
electrolytics and the non-polar 4.7u pair, A/C and A/K to 1/2 on the zeners
and LEDs (pad 1 is the cathode), TO-92 C,B,E to SOT-23 B,E,C, the dual-pitch
220p symbol's spare pad onto pad 2, the crystal's second pin onto 3225 pad 3,
and DIP-28 to TQFP-32 throughout IC7. Wires attach to pin positions, not pin
numbers, so this moves pads, not connections.

IC7 VCC/GND use KiCad 10 stacked pin numbers [4,6] and [3,5] so the TQFP's
second VCC and GND pads are connected as the datasheet requires. ADC6, ADC7
and the crystal's two case pads are new pads with no counterpart in the DIP
circuit; they are left unconnected, the crystal case pads pending a decision
on grounding them.

JP1-JP4, ISP0 and R28 keep their imported footprints: the connectors are
mechanically locked to the motherboard and the imported footprints are
anchored as the baseline board places them, and all six hand-soldered parts
are outside the JLC BOM. IC4 gets SOIC-16 but no LCSC field; the SSI2164 is
hand-soldered on arrival.

Verified with kicad-cli 10.0.6: the exported netlist is identical to the
baseline net for net under the pin remap, with only the six new pads added;
ERC reports the same 20 errors and 1 warning as the untouched baseline, with
six IC7 pins now named by their TQFP numbers. LCSC numbers, stock and
basic/extended status were read from JLC's parts API on 2026-09-16 and are
recorded with the substitution table in KiCad-SMD/README.md. No board work:
the .kicad_pcb is still the through-hole layout.

Co-Authored-By: Claude Opus 5 (1M context) <noreply@a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
Parts:
- C1, C27: footprint Voicecard-4P-v01-import-fps:ENP11-6.3 -> Capacitor_SMD:C_1206_3216Metric; LCSC (none) -> C29823
- C10, C21, C22, C9: footprint Voicecard-4P-v01-import-fps:C025-025X050 -> Capacitor_SMD:C_0603_1608Metric; LCSC (none) -> C107054
- C11, C12, C15, C16, C17, C18, C2, C20, C24, C28, C29, C3, C30, C5, C6, C8: footprint Voicecard-4P-v01-import-fps:C025-025X050 -> Capacitor_SMD:C_0603_1608Metric; LCSC (none) -> C14663
- C13, C19, C23, C7: footprint Voicecard-4P-v01-import-fps:C2.5_5-4 -> Capacitor_SMD:C_0603_1608Metric; LCSC (none) -> C106210
- C14, C25, C33: footprint Voicecard-4P-v01-import-fps:E2,5-6 -> Capacitor_SMD:CP_Elec_6.3x7.7; LCSC (none) -> C72477
- C26: footprint Voicecard-4P-v01-import-fps:C025-025X050 -> Capacitor_SMD:C_0603_1608Metric; LCSC (none) -> C21120
- C31, C32: footprint Voicecard-4P-v01-import-fps:C025-025X050 -> Capacitor_SMD:C_0603_1608Metric; LCSC (none) -> C1648
- C4: footprint Voicecard-4P-v01-import-fps:C025-025X050 -> Capacitor_SMD:C_0603_1608Metric; LCSC (none) -> C14858
- D1, D2: footprint Voicecard-4P-v01-import-fps:D-5 -> Diode_SMD:D_SOD-123; LCSC (none) -> C173412
- D3: footprint Voicecard-4P-v01-import-fps:D-5 -> Diode_SMD:D_SOD-123; LCSC (none) -> C173408
- IC1: footprint Voicecard-4P-v01-import-fps:DIL14 -> Package_SO:SOIC-14_3.9x8.7mm_P1.27mm; LCSC (none) -> C12594
- IC2: footprint Voicecard-4P-v01-import-fps:DIL16 -> Package_SO:SOIC-16_3.9x9.9mm_P1.27mm; LCSC (none) -> C174050
- IC3, IC5: footprint Voicecard-4P-v01-import-fps:DIL08 -> Package_SO:SOIC-8_3.9x4.9mm_P1.27mm; LCSC (none) -> C6961
- IC4: footprint Voicecard-4P-v01-import-fps:DIL16 -> Package_SO:SOIC-16_3.9x9.9mm_P1.27mm
- IC6: footprint Voicecard-4P-v01-import-fps:DIL08 -> Package_SO:SOIC-8_3.9x4.9mm_P1.27mm; LCSC (none) -> C16040
- IC7: footprint Voicecard-4P-v01-import-fps:DIL28-3 -> Package_QFP:TQFP-32_7x7mm_P0.8mm; LCSC (none) -> C14877
- LED1, LED2: footprint Voicecard-4P-v01-import-fps:LED3MM -> LED_SMD:LED_0805_2012Metric; LCSC (none) -> C84256
- Q1, Q2: footprint Voicecard-4P-v01-import-fps:TO92- -> Package_TO_SOT_SMD:SOT-23; LCSC (none) -> C53444
- Q3: footprint Voicecard-4P-v01-import-fps:HC49U-V -> Crystal:Crystal_SMD_3225-4Pin_3.2x2.5mm; LCSC (none) -> C255914
- R1, R12, R14: footprint Voicecard-4P-v01-import-fps:0204_7 -> Resistor_SMD:R_0603_1608Metric; LCSC (none) -> C4190
- R10, R11, R22, R23, R26, R27, R3, R4, R6, R7: footprint Voicecard-4P-v01-import-fps:0204_7 -> Resistor_SMD:R_0603_1608Metric; LCSC (none) -> C4216
- R13, R15, R16, R18, R2: footprint Voicecard-4P-v01-import-fps:0204_7 -> Resistor_SMD:R_0603_1608Metric; LCSC (none) -> C31850
- R17, R21, R34: footprint Voicecard-4P-v01-import-fps:0204_7 -> Resistor_SMD:R_0603_1608Metric; LCSC (none) -> C25804
- R19, R29, R32, R33: footprint Voicecard-4P-v01-import-fps:0204_7 -> Resistor_SMD:R_0603_1608Metric; LCSC (none) -> C22962
- R20, R24, R25, R30, R31, R5, R8, R9: footprint Voicecard-4P-v01-import-fps:0204_7 -> Resistor_SMD:R_0603_1608Metric; LCSC (none) -> C23179
Connections:
- net +5V: now also C33.1 (+), IC7.18 (AVCC), IC7.[4,6] (VCC); no longer C33.+, IC7.20 (AVCC), IC7.7 (VCC)
- net F_PWM: now also IC7.10 (PD6(AIN0)); no longer IC7.12 (PD6(AIN0))
- net GND: now also C14.2 (-), C25.1 (+), C33.2 (-), D3.1 (C), IC7.21 (GND), IC7.[3,5] (GND), LED1.1 (C), LED2.1 (C); no longer C14.-, C25.+, C33.-, D3.C, IC7.22 (GND), IC7.8 (GND), LED1.K (C), LED2.K (C)
- net I_GAIN: now also Q1.3 (C); no longer Q1.1 (C)
- net I_RESO: now also Q2.3 (C); no longer Q2.1 (C)
- net LP1: now also D1.2 (A); no longer C19.3, D1.A
- net LP2: no longer C7.3
- net LP3: no longer C13.3
- net LP4: now also C1.2; no longer C1.- (2), C23.3
- net MISO: now also IC7.16 (PB4(MISO)); no longer IC7.18 (PB4(MISO))
- net MOSI: now also IC7.15 (PB3(MOSI/OC2)); no longer IC7.17 (PB3(MOSI/OC2))
- net OSC: now also C27.2; no longer C27.- (2)
- net RES_PWM: now also IC7.9 (PD5(T1)); no longer IC7.11 (PD5(T1))
- net SCK: now also IC7.17 (PB5(SCK)); no longer IC7.19 (PB5(SCK))
- net SS: now also IC7.14 (PB2(SS/OC1B)); no longer IC7.16 (PB2(SS/OC1B))
- net VCC: now also C14.1 (+); no longer C14.+
- net VEE: now also C25.2 (-); no longer C25.-
- net at R14.2, R16.1: now also D3.2 (A); no longer D3.A
- net at R23.1: now also C27.1; no longer C27.+ (1)
- net at ISP0.5, R34.1: now also IC7.29 (PC6(/RESET)); no longer IC7.1 (PC6(/RESET))
- net at C15.2, IC1.1 (OUT): now also Q2.1 (B); no longer Q2.2 (B)
- net at R12.2: now also Q2.2 (E); no longer Q2.3 (E)
- net at C19.1, IC3.2 (-IN), IC4.4 (OUT): now also D2.2 (A); no longer D2.A
- net at C32.2, Q3.1: now also IC7.8 (PB7(XTAL2/TOSC2)); no longer IC7.10 (PB7(XTAL2/TOSC2))
- net at C2.2, IC1.14 (OUT): now also Q1.1 (B); no longer Q1.2 (B)
- net at R4.2: now also C1.1; no longer C1.+ (1)
- net at R31.1: now also LED2.2 (A); no longer LED2.A
- net at IC7.2 (PD4(XCK/T0)): now also IC6.3 (SCK)
- net at IC6.4 (SDI): now also IC7.31 (PD1(TXD)); no longer IC7.3 (PD1(TXD))
- net at IC6.2 (#CS): now also IC7.32 (PD2(INT0)); no longer IC7.4 (PD2(INT0))
- net at R30.1: now also LED1.2 (A); no longer LED1.A
- net at R1.2: now also Q1.2 (E); no longer Q1.3 (E)
- new net: C31.2, IC7.7 (PB6(XTAL1/TOSC1)), Q3.3 (2)
- new net: D1.1 (C), D2.1 (C)
- now unconnected: Q3.2

Commit message: Voicecard 4P SMD: ground the crystal case pads and clear the inherited ERC errors
Carey's decisions of 2026-09-16, applied in KiCad-SMD only so that ../KiCad/
keeps the imported baseline's ERC state.

The 3225's two case pads are grounded, which is the point of having them: they
are now one symbol pin with the stacked number [2,4], wired to the C31/C32
ground rail with a junction. The netlist shows Q3 pads 2 and 4 on GND.

The 20 ERC errors the Eagle import arrived with are annotation, not circuit
faults, so they are cleared to make a real error visible later: no-connect
flags on the 13 pins that are unused by design (IC7 AREF, PC0-PC3, PD0, PD3,
PD7, PB0, PB1; IC2 pins 2 and 15, the LM13700 diode-bias inputs; IC4 pin 1,
the 2164 MODE pin), and PWR_FLAGs on +5V, VCC, VEE and GND. The flags' value
text is hidden so it does not cover JP2's pin numbers.

PWR_FLAG is defined in a new project library, Voicecard-4P-SMD-extras.kicad_sym,
rather than taken from KiCad's global libraries, so the project stays
self-contained. It carries no footprint and does not appear in the BOM.

Two decisions confirmed with no file change: the 12 pF-load crystal stays,
with C31/C32 at 20p (two 20p in series plus stray lands at 12-14 pF, and no
value changes in Stage A), and R28 stays the through-hole 3296P.

Verified with kicad-cli 10.0.6: ERC is 0 errors and 1 warning, that warning
being IC2's unplaced buffer units A and B, which is inherent to using half an
LM13700. The netlist is still identical to the baseline net for net under the
pin remap, the BOM is unchanged at 87 components with no flag rows, and a PDF
render was checked for the new wiring and text overlap.

Co-Authored-By: Claude Opus 5 (1M context) <noreply@anthropic.com>
Connections:
- net GND: now also Q3.[2,4] (GND)
- no-connect marks 0 -> 13
